File: cube/cube.kicad_pcb (KiCad board)
At the start: 2 copper layers, 172.7 x 127 mm, 103 parts, among them J1 Conn_01x08, J10 Conn_01x08, J2 Conn_01x08, J3 Conn_01x08, J4 Conn_01x08, J5 Conn_01x08, J6 Conn_01x08, J7 Conn_01x08, J8 Conn_01x08, J9 Conn_01x08, Q1 PN2222A, Q2 PN2222A, Q3 PN2222A, Q4 PN2222A, Q5 PN2222A, Q6 PN2222A, Q7 PN2222A, Q8 PN2222A, U1 74HC595, U2 74HC595, U3 74HC595, U4 74HC595, U5 74HC595, U6 74HC595, U7 74HC595, U8 74HC595, U9 74HC595

Commit message: updated pcb.
Parts:
- added C10: 0.1uF, Capacitor_THT:C_Disc_D5.1mm_W3.2mm_P5.00mm, F.Cu at (49.6, 27.9)
- added C2: 0.1uF, Capacitor_THT:C_Disc_D5.1mm_W3.2mm_P5.00mm, F.Cu at (87.7, 27.9)
- added C3: 0.1uF, Capacitor_THT:C_Disc_D5.1mm_W3.2mm_P5.00mm, F.Cu at (49.6, 68.6)
- added C4: 0.1uF, Capacitor_THT:C_Disc_D5.1mm_W3.2mm_P5.00mm, F.Cu at (87.7, 68.6)
- added C5: 0.1uF, Capacitor_THT:C_Disc_D5.1mm_W3.2mm_P5.00mm, F.Cu at (49.6, 109.2)
- added C6: 0.1uF, Capacitor_THT:C_Disc_D5.1mm_W3.2mm_P5.00mm, F.Cu at (87.7, 109.2)
- added C7: 0.1uF, Capacitor_THT:C_Disc_D5.1mm_W3.2mm_P5.00mm, F.Cu at (125.8, 27.9)
- added C8: 0.1uF, Capacitor_THT:C_Disc_D5.1mm_W3.2mm_P5.00mm, F.Cu at (125.8, 68.6)
- added C9: 0.1uF, Capacitor_THT:C_Disc_D5.1mm_W3.2mm_P5.00mm, F.Cu at (142.2, 90.1)
Routing:
- net GND: track 568.4 -> 694.6 mm
- net +5V: track 439.5 -> 507.0 mm

Commit message: updated gerber files.
Parts:
- removed A1: Arduino_Nano_Every, Module:Arduino_Nano
- removed D1: LED, LED_THT:LED_D5.0mm_Clear
- removed J9: Conn_01x08, Connector_PinHeader_2.54mm:PinHeader_1x08_P2.54mm_Vertical
- removed R65: 220, Resistor_THT:R_Axial_DIN0207_L6.3mm_D2.5mm_P10.16mm_Horizontal
- added A2: SC0918, footprints:MODULE_SC0918, F.Cu at (165.6, 50.0)
- added C11: 0.33uF, Capacitor_THT:C_Disc_D5.1mm_W3.2mm_P5.00mm, F.Cu at (154.0, 88.6)
- added C12: 0.33uF, Capacitor_THT:C_Disc_D5.1mm_W3.2mm_P5.00mm, F.Cu at (173.0, 88.6)
- added D2: LED, LED_THT:LED_D5.0mm_Clear, F.Cu at (183.9, 50.8)
- added H1: MountingHole, MountingHole:MountingHole_3.2mm_M3_DIN965_Pad, F.Cu at (23.4, 28.2)
- added H2: MountingHole, MountingHole:MountingHole_3.2mm_M3_DIN965_Pad, F.Cu at (184.4, 28.2)
- added H3: MountingHole, MountingHole:MountingHole_3.2mm_M3_DIN965_Pad, F.Cu at (184.4, 145.8)
- added H4: MountingHole, MountingHole:MountingHole_3.2mm_M3_DIN965_Pad, F.Cu at (23.4, 145.8)
- added J11: Conn_01x08, Connector_PinHeader_2.54mm:PinHeader_1x08_P2.54mm_Vertical, F.Cu at (147.6, 45.5)
- added R74: 220, Resistor_THT:R_Axial_DIN0207_L6.3mm_D2.5mm_P10.16mm_Horizontal, F.Cu at (183.9, 34.5)
- added U10: L7805, Package_TO_SOT_THT:TO-220-3_Vertical, F.Cu at (163.3, 85.3)
- moved C9 14.5 mm to (137.4, 103.8)
- moved R70 14.5 mm to (145.0, 110.2)
- moved R73 14.5 mm to (155.2, 110.2)
- moved J10 14.5 mm to (142.5, 140.7)
- moved R66 14.5 mm to (170.4, 110.2)
- moved R67 14.5 mm to (165.4, 110.2)
- moved R68 14.5 mm to (134.9, 110.2)
- moved R69 14.5 mm to (140.0, 110.2)
- moved R71 14.5 mm to (150.1, 110.2)
- moved R72 14.5 mm to (160.3, 110.2)
- moved U9 14.5 mm to (142.5, 105.2)
- moved Q5 14.5 mm to (155.2, 128.0)
- moved Q1 14.5 mm to (124.7, 128.0)
- moved Q2 14.5 mm to (132.3, 128.0)
- moved Q3 14.5 mm to (140.0, 128.0)
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Routing:
- net LAYER_DATA: track 69.9 -> 34.8 mm
- net LAYER_LATCH: track 52.2 -> 25.9 mm
- net Net-(U3-QH'): track 109.9 -> 133.8 mm, vias 0 -> 1
- net LAYER_CLK: track 48.6 -> 29.5 mm
- net Net-(A1-A1): track 17.6 -> 0.00 mm
- net Net-(A1-SDA/A4): track 17.3 -> 0.00 mm
- net Net-(A1-A3): track 17.3 -> 0.00 mm
- net Net-(A1-A2): track 17.3 -> 0.00 mm
- net Net-(A1-SCL/A5): track 17.3 -> 0.00 mm
- net Net-(A1-A7): track 17.3 -> 0.00 mm
- net Net-(A1-A6): track 17.3 -> 0.00 mm
- net Net-(A1-A0): track 17.0 -> 0.00 mm
- net +5V: track 507.0 -> 518.6 mm
- net Net-(D1-A): track 11.2 -> 0.00 mm
- net VCC: track 0.00 -> 10.7 mm
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Other:
- board text added: "LED Cube - Strahinja Marinkovic, 2024"
- board text removed: "LED Cube - Strahinja Marinkovic, 2023"
